File: memori-hw/memori-hw.kicad_pcb (KiCad board)
At the start: 4 copper layers, 2 parts, among them J1 WeAct Studio 2.9" E-Paper Dis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, J2 Seeed Studio Xiao ESP32-C3

Commit message: feat(hw): Finished non-battery PCB.
Parts:
- moved J1 85.5 mm to (95.5, 97.8)
- moved J2 40.7 mm to (174.9, 101.7), turned to -90 degrees
Connections:
- net /GND renamed GND
Routing:
- net GND: track 0.00 -> 92.2 mm
- net /D/C: track 0.00 -> 91.9 mm
- net /BUSY: track 0.00 -> 85.6 mm
- net /CS: track 0.00 -> 85.5 mm
- net /3V3: track 0.00 -> 85.2 mm, vias 0 -> 2
- net /SDA: track 0.00 -> 83.2 mm
- net /SCL: track 0.00 -> 82.7 mm
- net /RES: track 0.00 -> 81.9 mm
Other:
- board outline added: 91.8 x 25.3 mm
- board text added: "MEM_C0RE"
- board text added: "Memento Mori."
- board text added: "Surendra J. Preston C. Cainan E. Julain M. Kenric T."
- board text added: "vFEB2026"

Commit message: feat(pcb): Finish memori PCB.
Parts:
- added R1: 220k, Resistor_THT:R_Axial_DIN0204_L3.6mm_D1.6mm_P7.62mm_Horizontal, F.Cu at (102.9, 93.7)
- added R2: 220k, Resistor_THT:R_Axial_DIN0204_L3.6mm_D1.6mm_P7.62mm_Horizontal, F.Cu at (102.9, 90.6)
- added U1: MOUDLE-SEEEDUINO-XIAO-ESP32C3, Seeed Studio XIAO Series Library:XIAO-ESP32C3-SMD, F.Cu at (174.9, 101.5)
- J2: value Seeed Studio Xiao ESP32-C3 -> Conn_01x02; footprint Seeed Studio XIAO Series Library:XIAO-ESP32C3-DIP -> Connector_JST:JST_PH_S2B-PH-K_1x02_P2.00mm_Horizontal
- moved J2 79.9 mm to (95.6, 111.7), turned to 90 degrees
Connections:
- J1 pad 5: /SCL -> /SCK
- J1 pad 6: /SDA -> /MOSI
- J2 pad 1: /D/C -> /BAT +
- J2 pad 2: /CS -> /BAT -
Routing:
- net /BAT -: track 0.00 -> 119.8 mm, vias 0 -> 3
- net /BAT +: track 0.00 -> 118.8 mm, vias 0 -> 3
- net /BATT_MONITOR: track 0.00 -> 92.9 mm, vias 0 -> 1
- net GND: track 92.2 -> 4.03 mm, vias 0 -> 1
- net /SDA: track 83.2 -> 0.00 mm
- net /SCL: track 82.7 -> 0.00 mm
- net /MOSI: track 0.00 -> 80.9 mm, vias 0 -> 2
- net /SCK: track 0.00 -> 80.0 mm, vias 0 -> 2
- net /BUSY: track 85.6 -> 80.0 mm, vias 0 -> 2
- net /RES: track 81.9 -> 79.4 mm, vias 0 -> 2
- net /D/C: track 91.9 -> 90.1 mm
- net /3V3: track 85.2 -> 83.5 mm, vias 2 -> 0
- net /CS: track 85.5 -> 83.9 mm
- added copper zone on F.Cu, net GND
Other:
- board text added: "+"
- board text added: "-"
- board text added: "3.7v Li-Po Battery"
- board text added: "CSE 115A Winter 2026 Surendra J. Preston C. Cainan E. Julian M. Kenric T."
- board text added: "Memento Mori"
- board text added: "Memori Mark-00"
- board text added: "The lone and level sands strech far away."
- board text added: "WeAct EPD 2.9{dblquote}"
- board text added: "Xiao ESP32C3"
- board text removed: "Memento Mori."
- board text removed: "Surendra J. Preston C. Cainan E. Julain M. Kenric T."
