File: memori-hw/memori-hw.kicad_sch (KiCad schematic)
At the start: 3 parts, among them J1 Conn_02x04_Odd_Even, J2 Conn_01x07, J3 Conn_01x07

Commit message: feat(hw): Finished with schematic.
Parts:
- removed J2, J3: Conn_01x07, symbol Connector_Generic:Conn_01x07
- added J2: Seeed Studio Xiao ESP32-C3, Seeed Studio XIAO Series Library:XIAO-ESP32C3-DIP, symbol Connector_Generic:Conn_02x07_Counter_Clockwise
- J1: value Conn_02x04_Odd_Even -> WeAct Studio 2.9{dblquote} E-Paper Display; footprint (none) -> Connector_PinHeader_2.54mm:PinHeader_2x04_P2.54mm_Vertical
Connections:
- net BUSY: now reaches J1.1 (Pin_1)
- net BUSY: now also J2.4 (Pin_4)
- net RES: now reaches J1.2 (Pin_2)
- net RES: now also J2.3 (Pin_3)
- net D/C: now reaches J1.3 (Pin_3)
- net D/C: now also J2.1 (GPIO2)
- net CS: now reaches J1.4 (Pin_4)
- net CS: now also J2.2 (Pin_2)
- net SCL: now reaches J1.5 (Pin_5)
- net SCL: now also J2.9 (Pin_9)
- net SDA: now reaches J1.6 (Pin_6)
- net SDA: now also J2.11 (Pin_11)
- net GND: now reaches J1.7 (Pin_7)
- net GND: now also J2.13 (Pin_13)
- net 3V3: now reaches J1.8 (Pin_8)
- net 3V3: now also J2.12 (Pin_12)
- no-connect marks 0 -> 6
Other:
- title: Mem_C0RE -> MEM_C0RE
- moved on the sheet: J1

Commit message: feat(hw): Finished non-battery PCB.
Changed lines of the file:
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@@
 	(wire
 		(pts
-			(xy 171.45 102.87) (xy 190.5 102.87)
+			(xy 171.45 102.87) (xy 198.12 102.87)
 		)
 		(stroke
@@
 			(width 0)
 			(type default)
-		)
-	)
-	(label "GND"
-		(at 190.5 102.87 0)
-		(effects
-			(font
-				(size 1.27 1.27)
-			)
-			(justify left bottom)
 		)
 	)
@@
 		)
 	)
-	(label "GND"
-		(at 72.39 113.03 180)
-		(effects
-			(font
-				(size 1.27 1.27)
-			)
-			(justify right bottom)
-		)
-	)
 	(label "RES"
 		(at 92.71 105.41 0)
@@
 			)
 			(justify right bottom)
+		)
+	)
+	(symbol
+		(lib_id "power:GND")
+		(at 198.12 102.87 0)
+		(unit 1)
+		(exclude_from_sim no)
+		(in_bom yes)
+		(on_board yes)
+		(dnp no)
+		(fields_autoplaced yes)
+		(property "Reference" "#PWR02"
+			(at 198.12 109.22 0)
+			(effects
+				(font
+					(size 1.27 1.27)
+				)
+				(hide yes)
+			)
+		)
+		(property "Value" "GND"
+			(at 198.12 107.95 0)
+			(effects
+				(font
+					(size 1.27 1.27)
+				)
+			)
+		)
+		(property "Footprint" ""
+			(at 198.12 102.87 0)
+			(effects
+				(font
+					(size 1.27 1.27)
+				)
+				(hide yes)
+			)
+		)
+		(property "Datasheet" ""
+			(at 198.12 102.87 0)
+			(effects
+				(font
+					(size 1.27 1.27)
+				)
+				(hide yes)
+			)
+		)
+		(property "Description" "Power symbol creates a global label with name \"GND\" , ground"
+			(at 198.12 102.87 0)
+			(effects
+				(font
+					(size 1.27 1.27)
+				)
+				(hide yes)
+			)
+		)
+		(pin "1"
+		)
+		(instances
+			(project "memori-hw"
+				(path "/81595af7-1809-407d-bce9-48813fee611e"
+					(reference "#PWR02")
+					(unit 1)
+				)
+			)
 		)
 	)
@@
 					(unit 1)
 				)
+			)
+		)
+	)
+	(symbol
+		(lib_id "power:GND")
+		(at 72.39 113.03 0)
+		(unit 1)
+		(exclude_from_sim no)
+		(in_bom yes)
+		(on_board yes)
+		(dnp no)
+		(fields_autoplaced yes)
+		(property "Reference" "#PWR01"
+			(at 72.39 119.38 0)
+			(effects
+				(font
+					(size 1.27 1.27)
+				)
+				(hide yes)
+			)
+		)
+		(property "Value" "GND"
+			(at 72.39 118.11 0)
+			(effects
+				(font
+					(size 1.27 1.27)
+				)
+			)
+		)
+		(property "Footprint" ""
+			(at 72.39 113.03 0)
+			(effects
+				(font
+					(size 1.27 1.27)
+				)
+				(hide yes)
+			)
+		)
+		(property "Datasheet" ""
+			(at 72.39 113.03 0)
+			(effects
+				(font
+					(size 1.27 1.27)
+				)
+				(hide yes)
+			)
+		)
+		(property "Description" "Power symbol creates a global label with name \"GND\" , ground"
+			(at 72.39 113.03 0)
+			(effects
+				(font
+					(size 1.27 1.27)
+				)
+				(hide yes)
+			)
+		)
+		(pin "1"
+		)
+		(instances
+			(project ""
+				(path "/81595af7-1809-407d-bce9-48813fee611e"
+					(reference "#PWR01")
+					(unit 1)
+				)

Commit message: feat(hw): Finished battery schematic.
Parts:
- removed J2: Seeed Studio Xiao ESP32-C3, Seeed Studio XIAO Series Library:XIAO-ESP32C3-DIP, symbol Connector_Generic:Conn_02x07_Counter_Clockwise
- added U1: MOUDLE-SEEEDUINO-XIAO-ESP32C3, Seeed Studio XIAO Series Library:XIAO-ESP32C3-SMD, symbol MOUDLE-SEEEDUINO-XIAO-ESP32C3:MOUDLE-SEEEDUINO-XIAO-ESP32C3
Connections:
- net 3V3: now also U1.12 (3V3)
- net BUSY: now also U1.5 (PA8_A4_D4_SDA)
- net CS: now also U1.3 (PA10_A2_D2)
- net D/C: now also U1.2 (PA4_A1_D1)
- net GND: now also U1.13 (GND)
- net RES: now also U1.4 (PA11_A3_D3)
- net SCL renamed SCK
- net SCK: now also U1.8 (PB09_A7_D7_RX)
- net SDA renamed MOSI
- net MOSI: now also U1.10 (PA5_A9_D9_MISO)
- no-connect marks 6 -> 11
Other:
- moved on the sheet: J1

Commit message: feat(pcb): Finish memori PCB.
Parts:
- added J2: Conn_01x02, Connector_JST:JST_PH_S2B-PH-K_1x02_P2.00mm_Horizontal, symbol Connector_Generic:Conn_01x02
- added R1, R2: 220k, Resistor_THT:R_Axial_DIN0204_L3.6mm_D1.6mm_P7.62mm_Horizontal, symbol Device:R
- J1: value WeAct Studio 2.9{dblquote} E-Paper Display -> WeAct Studio 2.9" E-Paper Display
Connections:
- net MOSI: now also U1.11 (PA6_A10_D10_MOSI); no longer U1.10 (PA5_A9_D9_MISO)
- net SCK: now also U1.9 (PA7_A8_D8_SCK); no longer U1.8 (PB09_A7_D7_RX)
- net BATT_MONITOR: now reaches U1.1 (PA02_A0_D0)
- net BATT_MONITOR: now also R1.1, R2.1
- net BAT +: now reaches U1.15 (BAT+)
- net BAT +: now also J2.1 (Pin_1), R1.2
- net BAT -: now reaches U1.16 (BAT-)
- net BAT -: now also J2.2 (Pin_2), R2.2
Other:
- note added: "+"
- note added: "-"
- moved on the sheet: J1
